File: hardware/pcb/pcb.kicad_pcb (KiCad board)
At the start: 2 copper layers, 121.8 x 86.2 mm, 25 parts, among them U1 YAAJ_BluePill_Part_Like_SWD_B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

Commit message: progres
Parts:
- added RV-LASER1: R_POT, Potentiometer_THT:Potentiometer_Piher_T-16H_Single_Horizontal, F.Cu at (158.9, 121.3)
- moved U-VLASER1 15.0 mm to (161.8, 108.9)
Connections:
- U-VLASER1 pad 2: Net-(J-LASER1-Pad1) -> Net-(RV-LASER1-Pad1)
Routing:
- net +12V: track 313.8 -> 338.4 mm, vias 7 -> 8
- net Net-(RV-LASER1-Pad1): track 0.00 -> 18.8 mm
- net GND: track 383.5 -> 399.5 mm
- net Net-(J-LASER1-Pad1): track 14.0 -> 21.5 mm
